File: Kicad/BTTS42Bv2/BTTS42Bv2.sch (KiCad schematic (older format))
At the start: 70 parts, among them K1-RES SW_Push, K2-Next SW_Push, K3-Mode SW_Push, K4-Valid SW_Push, P1 Conn_01x06, P2 Conn_01x04, P4 Conn_01x08, P5 Conn_01x02, U1 BNOR11, U2 A4950E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

Commit message: Fixed PCB designs
Parts:
- C1, C10: symbol Device:CP -> BTTS42Bv2-rescue:CP-Device
- C11, C12, C13, C14, C15, C16, C17, C18, C19, C2, C20, C21, C3, C4, C5, C6, C7, C8, C9: symbol Device:C -> BTTS42Bv2-rescue:C-Device
- D1, D4: symbol Device:LED -> BTTS42Bv2-rescue:LED-Device
- D2, D3, D5: symbol Device:D -> BTTS42Bv2-rescue:D-Device
- L1: renamed from L?; symbol pspice:INDUCTOR -> BTTS42Bv2-rescue:INDUCTOR-pspice
- Mode-K3: renamed from K3-Mode; symbol Switch:SW_Push -> BTTS42Bv2-rescue:SW_Push-Switch
- Next-K2: renamed from K2-Next; symbol Switch:SW_Push -> BTTS42Bv2-rescue:SW_Push-Switch
- P1: symbol Connector_Generic:Conn_01x06 -> BTTS42Bv2-rescue:Conn_01x06-Connector_Generic
- P2: symbol Connector_Generic:Conn_01x04 -> BTTS42Bv2-rescue:Conn_01x04-Connector_Generic
- P4: symbol Connector_Generic:Conn_01x08 -> BTTS42Bv2-rescue:Conn_01x08-Connector_Generic
- P5: symbol Connector_Generic:Conn_01x02 -> BTTS42Bv2-rescue:Conn_01x02-Connector_Generic
- R1, R10, R11, R12, R13, R14, R15, R16, R17, R18, R19, R2, R20, R21, R22, R23, R3, R5, R6, R7, R8, R9, R93: symbol Device:R -> BTTS42Bv2-rescue:R-Device
- RES-K1: renamed from K1-RES; symbol Switch:SW_Push -> BTTS42Bv2-rescue:SW_Push-Switch
- S1: symbol Switch:SW_DIP_x04 -> BTTS42Bv2-rescue:SW_DIP_x04-Switch
- U2, U4: symbol Driver_Motor:A4950E -> BTTS42Bv2-rescue:A4950E-Driver_Motor
- U7: symbol MCU_ST_STM32F1:STM32F103CBTx -> BTTS42Bv2-rescue:STM32F103CBTx-MCU_ST_STM32F1
- U8: symbol dk_PMIC-Voltage-Regulators-Linear:LD1117S33CTR -> BTTS42Bv2-rescue:LD1117S33CTR-dk_PMIC-Voltage-Regulators-Linear
- U9: symbol Interface_CAN_LIN:PCA82C251 -> BTTS42Bv2-rescue:PCA82C251-Interface_CAN_LIN
- Valid-K4: renamed from K4-Valid; symbol Switch:SW_Push -> BTTS42Bv2-rescue:SW_Push-Switch
- Y1: symbol Device:Crystal -> BTTS42Bv2-rescue:Crystal-Device
- p7: symbol Connector_Generic:Conn_01x07 -> BTTS42Bv2-rescue:Conn_01x07-Connector_Generic
Connections:
- net labels added: GND
- wire segments 164 -> 166
