File: Kicad/BTTS42Bv2/BTTS42Bv2.sch (KiCad schematic (older format))
At the start: 78 parts, among them P1 Conn_01x06, P2 Conn_01x04, P4 Conn_01x08, P5 Conn_01x02, U1 BNOR11, U2 A4950E, U3 EL-0631, U4 A4950E, U5 TLE5012B, U6 EL357NC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

Commit message: Merge remote-tracking branch 'origin/dev' into RevIngSchematics
# Conflicts:
#	.gitignore
#	Kicad/BTTS42Bv2/BTTS42Bv2-cache.lib
#	Kicad/BTTS42Bv2/BTTS42Bv2.sch
#	Kicad/BTTS42Bv2/BTT_S57B_v2.0_reverseIng.0.1.1.pdf
Connections:
- wire segments 170 -> 166
Changed lines of the file:
@@
 	9150 2450 9350 2450
-Wire Wire Line
-	8600 3000 9150 3000
 Wire Wire Line
 	9350 2450 9900 2450
 Connection ~ 9350 2450
-Wire Wire Line
-	8600 3100 9300 3100
 Wire Wire Line
 	9300 3100 9300 2600
@@
 	9600 2600 9900 2600
 Connection ~ 9600 2600
-	10350 5650 9950 5650
 $Comp
 L Mechanical:MountingHole_Pad H1
@@
 Wire Wire Line
 	2300 5900 2300 6050
-Wire Wire Line
-	9000 2450 9000 3000
-Wire Wire Line
-	9000 3000 8600 3000
-Wire Wire Line
-	9100 3100 8600 3100
-Wire Wire Line
-	9100 2600 9100 3100
 Text GLabel 9900 2800 0    50   Input ~ 0
 VDD
@@
 Text GLabel 10450 2800 2    50   Input ~ 0
 com
+Wire Wire Line
+	8600 3000 9150 3000
+Wire Wire Line
+	8600 3100 9300 3100
 $EndSCHEMATC
