File: Kicad/BTTS42Bv2/BTTS57Bv2.sch (KiCad schematic (older format))
At the start: 78 parts, among them P1 Conn_01x06, P2 Conn_01x04, P4 Conn_01x08, P5 Conn_01x02, U1 BNOR11, U2 A4950E, U3 EL-0631, U4 A4950E, U5 TLE5012B, U6 EL357NC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

Commit message: renamed files to S57B since schematics have CAN chips and only S57B has CAN bus
Parts:
- C1, C10: symbol BTTS42Bv2-rescue:CP-Device -> BTTS57Bv2-rescue:CP-Device
- C11, C12, C13, C14, C15, C16, C17, C18, C19, C2, C20, C21, C3, C4, C5, C6, C7, C8, C9: symbol BTTS42Bv2-rescue:C-Device -> BTTS57Bv2-rescue:C-Device
- D1, D4: symbol BTTS42Bv2-rescue:LED-Device -> BTTS57Bv2-rescue:LED-Device
- D2, D3, D5: symbol BTTS42Bv2-rescue:D-Device -> BTTS57Bv2-rescue:D-Device
- L1: symbol BTTS42Bv2-rescue:INDUCTOR-pspice -> BTTS57Bv2-rescue:INDUCTOR-pspice
- Mode-K3, Next-K2, RES-K1, Valid-K4: symbol BTTS42Bv2-rescue:SW_Push-Switch -> BTTS57Bv2-rescue:SW_Push-Switch
- P1: symbol BTTS42Bv2-rescue:Conn_01x06-Connector_Generic -> BTTS57Bv2-rescue:Conn_01x06-Connector_Generic
- P2: symbol BTTS42Bv2-rescue:Conn_01x04-Connector_Generic -> BTTS57Bv2-rescue:Conn_01x04-Connector_Generic
- P4: symbol BTTS42Bv2-rescue:Conn_01x08-Connector_Generic -> BTTS57Bv2-rescue:Conn_01x08-Connector_Generic
- P5: symbol BTTS42Bv2-rescue:Conn_01x02-Connector_Generic -> BTTS57Bv2-rescue:Conn_01x02-Connector_Generic
- R1, R10, R11, R12, R13, R14, R15, R16, R17, R18, R19, R2, R20, R21, R22, R23, R3, R5, R6, R7, R8, R9, R93: symbol BTTS42Bv2-rescue:R-Device -> BTTS57Bv2-rescue:R-Device
- S1: symbol BTTS42Bv2-rescue:SW_DIP_x04-Switch -> BTTS57Bv2-rescue:SW_DIP_x04-Switch
- U2, U4: symbol BTTS42Bv2-rescue:A4950E-Driver_Motor -> BTTS57Bv2-rescue:A4950E-Driver_Motor
- U7: symbol BTTS42Bv2-rescue:STM32F103CBTx-MCU_ST_STM32F1 -> BTTS57Bv2-rescue:STM32F103CBTx-MCU_ST_STM32F1
- U8: symbol BTTS42Bv2-rescue:LD1117S33CTR-dk_PMIC-Voltage-Regulators-Linear -> BTTS57Bv2-rescue:LD1117S33CTR-dk_PMIC-Voltage-Regulators-Linear
- U9: symbol BTTS42Bv2-rescue:PCA82C251-Interface_CAN_LIN -> BTTS57Bv2-rescue:PCA82C251-Interface_CAN_LIN
- Y1: symbol BTTS42Bv2-rescue:Crystal-Device -> BTTS57Bv2-rescue:Crystal-Device
- p7: symbol BTTS42Bv2-rescue:Conn_01x07-Connector_Generic -> BTTS57Bv2-rescue:Conn_01x07-Connector_Generic
